Commit message: [NEW]: 增加运动学插件及路径规划算法对比测试
增加运动学插件及路径规划算法对比测试文件
增加对上述测试结果的分析与输出

File: src/russ_description/urdf/russ.urdf (robot description, URDF)
Before this commit: robot russ, 13 links, 12 joints
Links:
- link base_link: geometry collision mesh filename=package://russ_description/meshes/arm_base_link.STL; visual mesh filename=package://russ_description/meshes/base.dae
- link forearm_link: geometry collision mesh filename=package://russ_description/meshes/forearm_link.STL; visual mesh filename=package://russ_description/meshes/forearm.dae
- link kinect_link: geometry collision mesh filename=package://russ_description/meshes/camera_link.STL; visual mesh filename=package://russ_description/meshes/kinect.dae
- link shoulder_link: geometry collision mesh filename=package://russ_description/meshes/shoulder_link.STL; visual mesh filename=package://russ_description/meshes/shoulder.dae
- link upperarm_link: geometry collision mesh filename=package://russ_description/meshes/upperarm_link.STL; visual mesh filename=package://russ_description/meshes/upperarm.dae
- link wrist1_link: geometry collision mesh filename=package://russ_description/meshes/wrist1_link.STL; visual mesh filename=package://russ_description/meshes/wrist1.dae
- link wrist2_link: geometry collision mesh filename=package://russ_description/meshes/wrist2_link.STL; visual mesh filename=package://russ_description/meshes/wrist2.dae
- link wrist3_link: geometry collision mesh filename=package://russ_description/meshes/wrist3_link.STL; visual mesh filename=package://russ_description/meshes/wrist3.dae
