Commit message: [NEW]: 添加人体urdf模型

File: src/russ_description/urdf/russ_man.urdf (robot description, URDF)
Before this commit: robot russ, 13 links, 12 joints
Links:
- added link man_link, mass 58.24; collision mesh filename=package://russ_description/meshes/man/man_link.STL; visual mesh filename=package://russ_description/meshes/man/man_link.STL
- added link upperprobe_link, mass 0.29224119341871; collision mesh filename=package://russ_description/meshes/man/upperprobe_link.STL; visual mesh filename=package://russ_description/meshes/man/upperprobe_link.STL
- link base_link: geometry collision mesh filename=package://russ_description/meshes/man/arm_base_link.STL; visual mesh filename=package://russ_description/meshes/man/base.dae
- link bed_link: geometry collision mesh filename=package://russ_description/meshes/man/bed_link.STL; visual mesh filename=package://russ_description/meshes/man/bed_link.STL
- link camera_holder_link: mass 10.767 -> 10.7674813244167; geometry collision mesh filename=package://russ_description/meshes/man/camera_holder_link.STL; visual mesh filename=package://russ_description/meshes/man/camera_holder_link.STL
- link forearm_link: geometry collision mesh filename=package://russ_description/meshes/man/forearm_link.STL; visual mesh filename=package://russ_description/meshes/man/forearm.dae
- link kinect_link: geometry collision mesh filename=package://russ_description/meshes/man/camera_link.STL; visual mesh filename=package://russ_description/meshes/man/camera_link.STL
- link probe_link: mass 0.31983 -> 0.0275873695177772; geometry collision mesh filename=package://russ_description/meshes/man/probe_link.STL; visual mesh filename=package://russ_description/meshes/man/probe_link.STL
- link shoulder_link: geometry collision mesh filename=package://russ_description/meshes/man/shoulder_link.STL; visual mesh filename=package://russ_description/meshes/man/shoulder.dae
- link table_base_link: mass 309.143354179708 -> 309.14; geometry collision mesh filename=package://russ_description/meshes/man/base_link.STL; visual mesh filename=package://russ_description/meshes/man/base_link.STL
- link upperarm_link: geometry collision mesh filename=package://russ_description/meshes/man/upperarm_link.STL; visual mesh filename=package://russ_description/meshes/man/upperarm.dae
- link wrist1_link: geometry collision mesh filename=package://russ_description/meshes/man/wrist1_link.STL; visual mesh filename=package://russ_description/meshes/man/wrist1.dae
- link wrist2_link: geometry collision mesh filename=package://russ_description/meshes/man/wrist2_link.STL; visual mesh filename=package://russ_description/meshes/man/wrist2.dae
- link wrist3_link: geometry collision mesh filename=package://russ_description/meshes/man/wrist3_link.STL; visual mesh filename=package://russ_description/meshes/man/wrist3.dae
Joints:
- added joint man_joint: type fixed, parent bed_link, child man_link, origin xyz=0.466 -0.074751 0.19344 rpy=0 0 0, axis 0 0 0
- added joint upperprobe_joint: type fixed, parent wrist3_link, child upperprobe_link, origin xyz=0 0.1086 0 rpy=0 0 0, axis 0 0 0
- joint base_joint: origin xyz=0 0.37 0.7002 rpy=0 0 0 -> xyz=0 0.37 0.7 rpy=0 0 0
- joint camera_holder_joint: origin xyz=0 1.3832 1.4643 rpy=3.1416 0.5236 1.5708 -> xyz=0 1.3665 1.4643 rpy=3.1416 0.5236 1.5708
- joint forearm_joint: limit lower=-3.14159265 upper=3.14159265 effort=150 velocity=3.15 -> lower=-3.1416 upper=3.1416 effort=150 velocity=3.15
- joint kinect_joint: origin xyz=-0.05355 -0.0021296 0.016187 rpy=0 -1.5708 0 -> xyz=-0.0535 -0.00026386 0.011407 rpy=-1.8978 -1.5708 1.9025
- joint probe_joint: origin xyz=0 0.268599999411803 0 rpy=0 0 0 -> xyz=0 0.16 0 rpy=0 0 0; parent wrist3_link -> upperprobe_link
- joint shoulder_joint: limit lower=-3.14159265 upper=3.14159265 effort=150 velocity=3.15 -> lower=-3.1416 upper=3.1416 effort=150 velocity=3.15; origin xyz=0 0 0.1623 rpy=0 0 0 -> xyz=0 0 0.1625 rpy=0 0 0
- joint upperarm_joint: limit lower=-3.14159265 upper=3.14159265 effort=150 velocity=3.15 -> lower=-3.1416 upper=3.1416 effort=150 velocity=3.15
- joint wrist1_joint: limit lower=-3.14159265 upper=3.14159265 effort=28 velocity=3.2 -> lower=-3.1416 upper=3.1416 effort=28 velocity=3.2
- joint wrist2_joint: limit lower=-3.14159265 upper=3.14159265 effort=28 velocity=3.2 -> lower=-3.1416 upper=3.1416 effort=28 velocity=3.2

Commit message: [WIP]: 增加对心脏部位扫查的测试文件
增加对心脏部位waypoint自动扫查的测试文件
由于机械臂Link与man_link的碰撞检测存在未知问题，
暂时增加了对upperarm_link的运动限位

File: src/russ_description/urdf/russ_man.urdf (robot description, URDF)
Before this commit: robot russ, 15 links, 14 joints
Joints:
- joint upperarm_joint: limit lower=-3.1416 upper=3.1416 effort=150 velocity=3.15 -> lower=-1.4137 upper=1.4137 effort=150 velocity=3.15

Commit message: [FIX]: 修正机械臂link与man碰撞检测问题
修正russ_man_moveit启动配置，将russ_moveit修正为russ_man_moveit
因规划可检测机械臂与man碰撞，故原有upperarm_joint限位取消

File: src/russ_description/urdf/russ_man.urdf (robot description, URDF)
Before this commit: robot russ, 15 links, 14 joints
Joints:
- joint upperarm_joint: limit lower=-1.4137 upper=1.4137 effort=150 velocity=3.15 -> lower=-3.1416 upper=3.1416 effort=150 velocity=3.15
